File: Production/SCD40/SparkFun_Qwiic_CO2_Sensor_SCD40-Panel.brd (EAGLE design)
At the start: 175 x 117.3 mm, 1134 parts, among them J1 QWIIC_RA, J10 QWIIC_RA, J11 QWIIC_RA, J12 PTH, J13 QWIIC_RA, J14 QWIIC_RA, J15 PTH, J16 QWIIC_RA, J17 QWIIC_RA, J18 PTH, J19 QWIIC_RA, J2 QWIIC_RA, J20 QWIIC_RA, J21 PTH, J22 QWIIC_RA, J23 QWIIC_RA, J24 PTH, J25 QWIIC_RA, J26 QWIIC_RA, J27 PTH, J28 QWIIC_RA, J29 QWIIC_RA, J3 PTH, J30 PTH, J31 QWIIC_RA, J32 QWIIC_RA, J33 PTH, J34 QWIIC_RA, J35 QWIIC_RA, J36 PTH, J37 QWIIC_RA, J38 QWIIC_RA, J39 PTH, J4 QWIIC_RA, J40 QWIIC_RA, J41 QWIIC_RA, J42 PTH, J43 QWIIC_RA, J44 QWIIC_RA, J45 PTH, J46 QWIIC_RA, J47 QWIIC_RA, J48 PTH, J49 QWIIC_RA, J5 QWIIC_RA, J50 QWIIC_RA, J51 PTH, J52 QWIIC_RA, J53 QWIIC_RA, J54 PTH, J55 QWIIC_RA, J56 QWIIC_RA, J57 PTH, J58 QWIIC_RA, J59 QWIIC_RA, J6 PTH, J60 PTH, J61 QWIIC_RA, J62 QWIIC_RA, J63 PTH, J64 QWIIC_RA, J65 QWIIC_RA, J66 PTH, J67 QWIIC_RA, J68 QWIIC_RA, J69 PTH, J7 QWIIC_RA, J70 QWIIC_RA, J71 QWIIC_RA, J72 PTH, J8 QWIIC_RA, J9 PTH, U1 SCD40/1, U10 SCD40/1, U11 SCD40, U12 SCD41, U13 SCD40/1, U14 SCD40, U15 SCD41, U16 SCD40/1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

Commit message: Update from pre-design review notes.
Changed I2C PURs from 4.7k to 2.2k to match Qwiic standards.
Changed wording on revision.
Update top stop of pin 1 of sensor.
Repanelize.
Parts:
- R1, R10, R11, R13, R14, R16, R17, R19, R2, R20, R22, R23, R25, R26, R28, R29, R31, R32, R34, R35, R37, R38, R4, R40, R41, R43, R44, R46, R47, R49, R5, R50, R52, R53, R55, R56, R58, R59, R61, R62, R64, R65, R67, R68, R7, R70, R71, R8: value 4.7k -> 2.2k
